Commit message: remove transmision tags & base link,fix location

File: desc/b1_box_collide.urdf (robot description, URDF)
Before this commit: robot b1_description, 31 links, 30 joints
Links:
- removed link base
Joints:
- removed joint floating_base

File: desc/b1_mesh_collide.urdf (robot description, URDF)
Before this commit: robot b1_description, 31 links, 30 joints
Links:
- removed link base
- link FL_calf: geometry collision mesh filename=/meshes/calf.dae scale=1 1 1; visual mesh filename=/meshes/calf.dae scale=1 1 1
- link FL_hip: geometry collision mesh filename=/meshes/hip.dae scale=1 1 1; visual mesh filename=/meshes/hip.dae scale=1 1 1
- link FL_thigh: geometry collision mesh filename=/meshes/thigh.dae scale=1 1 1; visual mesh filename=/meshes/thigh.dae scale=1 1 1
- link FR_calf: geometry collision mesh filename=/meshes/calf.dae scale=1 1 1; visual mesh filename=/meshes/calf.dae scale=1 1 1
- link FR_hip: geometry collision mesh filename=/meshes/hip.dae scale=1 1 1; visual mesh filename=/meshes/hip.dae scale=1 1 1
- link FR_thigh: geometry collision mesh filename=/meshes/thigh_mirror.dae scale=1 1 1; visual mesh filename=/meshes/thigh_mirror.dae scale=1 1 1
- link RL_calf: geometry collision mesh filename=/meshes/calf.dae scale=1 1 1; visual mesh filename=/meshes/calf.dae scale=1 1 1
- link RL_hip: geometry collision mesh filename=/meshes/hip.dae scale=1 1 1; visual mesh filename=/meshes/hip.dae scale=1 1 1
- link RL_thigh: geometry collision mesh filename=/meshes/thigh.dae scale=1 1 1; visual mesh filename=/meshes/thigh.dae scale=1 1 1
- link RR_calf: geometry collision mesh filename=/meshes/calf.dae scale=1 1 1; visual mesh filename=/meshes/calf.dae scale=1 1 1
- link RR_hip: geometry collision mesh filename=/meshes/hip.dae scale=1 1 1; visual mesh filename=/meshes/hip.dae scale=1 1 1
- link RR_thigh: geometry collision mesh filename=/meshes/thigh_mirror.dae scale=1 1 1; visual mesh filename=/meshes/thigh_mirror.dae scale=1 1 1
Joints:
- removed joint floating_base

File: desc/xacro/b1_box_collide.xacro (robot description, xacro)
@@ -19,5 +19,5 @@
         </joint>
     </xacro:if>  -->
-    <link name="base">
+    <!-- <link name="base">
         <visual>
             <origin rpy="0 0 0" xyz="0 0 0"/>
@@ -31,5 +31,5 @@
         <parent link="base"/>
         <child link="trunk"/>
-    </joint>
+    </joint> -->
     <link name="trunk">
         <visual>

File: desc/xacro/b1_mesh_collide.xacro (robot description, xacro)
@@ -6,5 +6,5 @@
     <xacro:include filename="const.xacro"/>
     <xacro:include filename="materials.xacro"/>
-    <xacro:include filename="leg.xacro"/>
+    <xacro:include filename="leg_mesh_collision.xacro"/>
     <!-- <xacro:include filename="$(find b1_description)/xacro/gazebo.xacro"/> -->
     <!-- Rotor related joint and link is only for demonstrate location. -->
@@ -19,5 +19,5 @@
         </joint>
     </xacro:if>  -->
-    <link name="base">
+    <!-- <link name="base">
         <visual>
             <origin rpy="0 0 0" xyz="0 0 0"/>
@@ -31,5 +31,5 @@
         <parent link="base"/>
         <child link="trunk"/>
-    </joint>
+    </joint> -->
     <link name="trunk">
         <visual>

File: desc/xacro/leg.xacro (robot description, xacro)
@@ -1,5 +1,5 @@
 <?xml version="1.0"?>
 <robot xmlns:xacro="http://www.ros.org/wiki/xacro">
-    <xacro:include filename="transmission.xacro"/>
+    <!-- <xacro:include filename="transmission.xacro"/> -->
     <xacro:macro name="leg" params="name mirror mirror_dae front_hind front_hind_dae">
         <joint name="${name}_hip_joint" type="revolute">
@@ -250,5 +250,5 @@
             </inertial>
         </link>
-        <xacro:leg_transmission name="${name}"/>
+        <!-- <xacro:leg_transmission name="${name}"/> -->
     </xacro:macro>
 </robot>

File: desc/xacro/transmission.xacro (robot description, xacro)
@@ -1,3 +1,3 @@
-<?xml version="1.0"?>
+<!-- <?xml version="1.0"?>
 <robot xmlns:xacro="http://www.ros.org/wiki/xacro">
     <xacro:macro name="leg_transmission" params="name">
@@ -6,5 +6,5 @@
             <joint name="${name}_hip_joint">
             <hardwareInterface>hardware_interface/EffortJointInterface</hardwareInterface>
-            </joint>
+            </jointf>
             <actuator name="${name}_hip_motor">
             <hardwareInterface>hardware_interface/EffortJointInterface</hardwareInterface>
@@ -33,3 +33,3 @@
         </transmission>
     </xacro:macro>
-</robot>
+</robot> -->
